Commit message: [Project] adding robotic arm link and joints

File: course_2_hardwareSimulation/urdf/common_properties.xacro (robot description, xacro)
@@ -9,4 +9,10 @@
     <material name="grey">
         <color rgba="0.1 0.1 0.1 1" />
+    </material>
+    <material name="yellow">
+        <color rgba="0.5 0.5 0.0 1" />
+    </material>
+    <material name="orange">
+        <color rgba="0.7 0.4 0.0 1" />
     </material>
     <xacro:macro name="inertia_box" params="l w h m xyz rpy">

Commit message: fixing interial tag for box macro which was preventing the robot arm to spawn in gazebo

File: course_2_hardwareSimulation/urdf/common_properties.xacro (robot description, xacro)
@@ -16,6 +16,6 @@
         <color rgba="0.7 0.4 0.0 1" />
     </material>
-    <xacro:macro name="inertia_box" params="l w h m xyz rpy">
-        <inertail>
+    <xacro:macro name="inertia_box" params="m l w h xyz rpy">
+        <inertial>
             <origin xyz="${xyz}" rpy="${rpy}" />
             <mass value="${m}" />
@@ -23,7 +23,7 @@
                 iyy="${(m/12)*(w*w + l*l)}" iyz="0"
                 izz="${(m/12)*(h*h + w*w)}" />
-        </inertail>
+        </inertial>
     </xacro:macro>
-    <xacro:macro name="inertia_cylinder" params="r h m xyz rpy">
+    <xacro:macro name="inertia_cylinder" params="m r h xyz rpy">
         <inertial>
             <origin xzy="${xyz}" rpy="${rpy}" />

File: course_2_hardwareSimulation/urdf/my_robot.urdf.xacro (robot description, xacro)
@@ -3,5 +3,5 @@
     <xacro:include filename="common_properties.xacro"/>
     <!-- the included files can be used in the other include files as well -->
-    <xacro:include filename="mobile_base.xacro"/>
+    <xacro:include filename="mobile_base_2.xacro"/>
     <xacro:include filename="camera.xacro"/>
     <xacro:include filename="mobile_base_gazebo.xacro"/>
