Commit message: [Project]: finished final project with robot base and hand

File: course_2_hardwareSimulation/urdf/arm.xacro (robot description, xacro)
@@ -57,4 +57,5 @@
         <axis xyz="0 1 0" />
         <limit lower="0.0" upper="${pi/2.0}" effort="100.0" velocity="100.0" />
+        <dynamics friction="0.05" damping="0.1" />
     </joint>
     <xacro:arm_link prefix="hand" color="orange" />
@@ -65,4 +66,5 @@
         <axis xyz="0 1 0" />
         <limit lower="0.0" upper="${pi/2.0}" effort="100.0" velocity="100.0" />
+        <dynamics friction="0.05" damping="0.1" />
     </joint>
 </robot>

File: course_2_hardwareSimulation/urdf/arm_gazebo.xacro (robot description, xacro)
@@ -10,3 +10,17 @@
         <material>Gazebo/Orange</material>
     </gazebo>
+    <gazebo>
+        <plugin name="joint_state_publisher_controller"
+            filename="libgazebo_ros_joint_state_publisher.so">
+            <update_rate>10</update_rate>
+            <joint_name>base_forearm_joint</joint_name>
+            <joint_name>forearm_hand_joint</joint_name>
+        </plugin>
+    </gazebo>
+    <gazebo>
+        <plugin name="joint_pose_trajectory_controller"
+            filename="libgazebo_ros_joint_pose_trajectory.so">
+            <update_rate>2</update_rate>
+        </plugin>
+    </gazebo>
 </robot>

File: course_2_hardwareSimulation/urdf/mobile_base.xacro (robot description, xacro)
@@ -85,7 +85,7 @@
     </link>
     <joint name="base_baseFootprint_jt" type="fixed">
-        <parent link="base_link" />
-        <child link="base_footprint" />
-        <origin xyz="0 0 ${-wheel_radius}" rpy="0 0 0" />
+        <parent link="base_footprint" />
+        <child link="base_link" />
+        <origin xyz="0 0 ${wheel_radius}" rpy="0 0 0" />
     </joint>
 </robot>

File: course_2_hardwareSimulation/urdf/my_robot.urdf.xacro (robot description, xacro)
@@ -3,6 +3,13 @@
     <xacro:include filename="common_properties.xacro"/>
     <!-- the included files can be used in the other include files as well -->
-    <xacro:include filename="mobile_base_2.xacro"/>
-    <xacro:include filename="camera.xacro"/>
+    <xacro:include filename="arm.xacro" />
+    <xacro:include filename="mobile_base.xacro"/>
+    <!-- <xacro:include filename="camera.xacro"/> -->
+    <xacro:include filename="arm_gazebo.xacro" />
     <xacro:include filename="mobile_base_gazebo.xacro"/>
+    <joint name="base_arm_jt" type="fixed">
+        <parent link="base_link" />
+        <child link="arm_base_link" />
+        <origin xyz="${base_length / 4} 0 ${base_height}" rpy="0 0 0" />
+    </joint>
 </robot>
